Commit message: Add Gazebo simulation

File: dh_description/urdf/ag95/base_link.urdf.xacro (robot description, xacro)
@@ -18,13 +18,13 @@
         </geometry>
       </collision>
+      <inertial>
+        <origin xyz="-1.9172E-05 4.6267E-05 0.054522" rpy="0 0 0" />
+        <mass value="0.3499" />
+        <inertia
+          ixx="0.00050797" ixy="6.5338E-08" ixz="-7.1191E-08"
+          iyy="0.00038427" iyz="3.8152E-07"
+          izz="0.00016523" />
+      </inertial>
     </link>
-    <inertial>
-      <origin xyz="-1.9172E-05 4.6267E-05 0.054522" rpy="0 0 0" />
-      <mass value="0.3499" />
-      <inertia
-        ixx="0.00050797" ixy="6.5338E-08" ixz="-7.1191E-08"
-        iyy="0.00038427" iyz="3.8152E-07"
-        izz="0.00016523" />
-    </inertial>
   </xacro:macro>
 </robot>

File: dh_description/urdf/ag95_gripper.urdf.xacro (robot description, xacro)
@@ -3,5 +3,7 @@
   <xacro:include filename="$(find dh_description)/urdf/ag95.urdf.xacro" />
   <xacro:include filename="$(find dh_description)/urdf/ag95/finger.transmission.xacro" />
-  <xacro:ag95 prefix="ag95_" />
-  <xacro:finger_transmission prefix="ag95_" mechanical_reduction="${-100/0.03}" />
+  <xacro:include filename="$(find dh_description)/urdf/ag95.gazebo.xacro" />
+  <xacro:ag95 prefix="ag95_"/>
+  <xacro:finger_transmission prefix="ag95_" mechanical_reduction="${-100/0.03}"/>
+  <xacro:ag95_gazebo prefix="ag95_" ns="/dh_ag95"/>
 </robot>
